File: high_altitude_balloon.kicad_sch (KiCad schematic)
At the start: 0 parts

Commit message: real schematic with all components placed
Parts:
- added C1, C2, C3, C4, C5, C6, C7, C8, C9: C, symbol Device:C
- added D1, D2, D3: LED, symbol Device:LED
- added J1: USB_C_Receptacle_USB2.0_16P, symbol Connector:USB_C_Receptacle_USB2.0_16P
- added J2, J4: Conn_01x04, symbol Connector_Generic:Conn_01x04
- added J3: Conn_01x06, symbol Connector_Generic:Conn_01x06
- added J5: Conn_01x05, symbol Connector_Generic:Conn_01x05
- added J6: SD_Card_Device, symbol Connector:SD_Card_Device
- added J7: Conn_01x02, symbol Connector_Generic:Conn_01x02
- added R1, R2, R3, R4, R5, R6: R, symbol Device:R
- added SW1: SW_Push, symbol Switch:SW_Push
- added TP1, TP2, TP3, TP4, TP5, TP6: TestPoint, symbol Connector:TestPoint
- added U1: MSPM0G3507SRGZR, RGZ0048A-IPC_A, symbol correct_mcu:MSPM0G3507SRGZR
- added U2: CP2102N-Axx-xQFN20, Package_DFN_QFN:SiliconLabs_QFN-20-1EP_3x3mm_P0.5mm, symbol Interface_USB:CP2102N-Axx-xQFN20
- added U3: XC6206PxxxMR, Package_TO_SOT_SMD:SOT-23-3, symbol Regulator_Linear:XC6206PxxxMR
- added U4: RFM95W-915S2, symbol RF_Module:RFM95W-915S2
- added U5: BME680, Package_LGA:Bosch_LGA-8_3x3mm_P0.8mm_ClockwisePinNumbering, symbol Sensor:BME680
- added Y1: Crystal, symbol Device:Crystal
Connections:
- new net: J1.A1 (GND), J1.A12 (GND), J1.B1 (GND), J1.B12 (GND)
- new net: J1.A4 (VBUS), J1.A9 (VBUS), J1.B4 (VBUS), J1.B9 (VBUS)
- new net: U2.12 (GND), U2.21 (GND), U2.3 (GND)
- new net: J6.3 (VSS), J6.6 (VSS)
Other:
- note added: "EXTERNAL OUTPUTS"
- note added: "HEADER PINS FOR CONNECTION"
- note added: "LORA AND TEMP SENSOR"
- note added: "Microcontroller"
- note added: "PASSIVE COMPONENTS"
- note added: "TIMING, RESET AND DEBUG"
- note added: "Test Points: So we know each segment is working"
