File: pcb/v1/328.kicad_sch (KiCad schematic)
At the start: 37 parts, among them J1 USB_C_Receptacle_USB2.0_16P, J2 CONNECTS TO GPS, J3 LiPo Connection, J5 Conn_01x05, J6 SD_Card_Device, SW1 SW_Push, U1 MSPM0G3507SRGZR, U2 USB TO UART, U3 Low Dropout Regulator, U4 RFM95W-915S2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

Commit message: pcb updates
Parts:
- removed L1: L, Inductor_SMD:L_0402_1005Metric, symbol Device:L
